File: 08_kicad_flow_work/led_circuit_v1/led_circuit_v1.kicad_pcb (KiCad board)
At the start: 2 copper layers, 79 x 32 mm, 4 parts, among them SW1 SW_DPST_x2

Commit message: practica 09: diseño de fuente de poder
Other:
- board text added: "By:Gilbert"
Changed lines of the file:
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@@
 		(layer "Edge.Cuts")
+	)
+	(gr_text "By:Gilbert"
+		(at 202 100 0)
+		(layer "B.SilkS")
+		(effects
+			(font
+				(size 2 2)
+				(thickness 0.3)
+			)
+			(justify mirror)
+		)
 	)
 	(segment
